Commit message: 1. allegro hand urdf modification into neuralfeels convetion 2. new task env defined for contact maximization

File: assets/allegro/allegro_digit_left_elastomer.urdf (robot description, URDF)
Before this commit: robot allegro_hand_left_digit_elastomer, 25 links, 24 joints
Joints:
- joint joint_13_0: origin xyz=-0.027 0.005 0.0399 -> xyz=-0.027 -0.005 0.0399
- joint joint_15_0_tip: origin xyz=0 0 0.0303 rpy=0 0 0 -> xyz=0 0 0.0303 rpy=0 0 1.047
